File: Design/H2BR1.sch (EAGLE design)
At the start: 30 parts, among them P1 HEXABIT_17.32_NO_P6_P7_P12, U1 STM32G0B1CEU6NUFQFPN48_STM32_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, U2 LD39015M18RSOT23-5L_STM-L, U3 MAX30100EFD+, X1 XTALL_CSTCE8M00G52

Commit message: -The final design, all done.
Parts:
- removed INT, SCL, SDA: PAD1, HEXABITZ_CONNECTION_PARTS:PAD4
- added C13: 1uF, HEXABITZ_RCLS:C-0805
- added C14: 10uF, HEXABITZ_RCLS:C-0805
- added D2: BOURNS_CDSOD323-T03SCBOURNS_CDSOD323-T03SC_0_0, HEXABITZ_RCLS:BOURNS_CDSOD323-T03SCBOURNS_CDSOD323-T03SC_0_0
- added L1: ASMPH08062R2MT, HEXABITZ_RCLS:ASMPH08062R2MT
- added R10, R9: 0R, HEXABITZ_RCLS:R-0603
- added R7: 750K, HEXABITZ_RCLS:R-0603
- added R8: 100K, HEXABITZ_RCLS:R-0603
- added TRIMBLE-LOGO1: HEXA-LOGO, HEXABITZ_USER_INTERFACE_PARTS:HEXA-LOGO
- added U4: PAM2401YPADJ, HEXABITZ_ICs:PAM2401YPADJ
- C10: value 10uF -> 22uF; device HEXABITZ_RCLS:T491A106K010AT -> HEXABITZ_RCLS:C-0603
- C11: value 10uF -> 22pF; device HEXABITZ_RCLS:T491A106K010AT -> HEXABITZ_RCLS:C-0603; STATUS (none) -> DNP
- C12: value 100nF -> 10uF; device HEXABITZ_RCLS:C-0603 -> HEXABITZ_RCLS:C-0805
- C2, C4: device HEXABITZ_RCLS:C-0805-POL -> HEXABITZ_RCLS:C-0805
- C7: value 4.7uF -> 10uF; device HEXABITZ_RCLS:C-0805-POL -> HEXABITZ_RCLS:C-0805
- C8: value 100nF -> 4.7uF; device HEXABITZ_RCLS:C-0603 -> HEXABITZ_RCLS:C-0805
- D1: value VLMS1300-GS08 -> RED
- FB1: device HEXABITZ_RCLS:FB-TDK_MMZ1608Y300B -> HEXABITZ_RCLS:FB-0603
- R4, R5, R6: value 4.7K -> 1K
- U1: value STM32G0B1CEU6NUFQFPN48_STM32_STM -> STM32G0B1CEU6QFN_B1CEU6_STM-L; device HEXABITZ_ICs:STM32G0B1CEU6NUFQFPN48_STM32_STM -> HEXABITZ_ICs:STM32G0B1CEU6QFN_B1CEU6_STM-L
- U2: value LD39015M18RSOT23-5L_STM-L -> LDK130PU18R; device HEXABITZ_ICs:LD39015M18RSOT23-5L_STM-L -> HEXABITZ_ICs:LDK130PU18R
- U3: value MAX30100EFD+ -> MAX30101EFD+T; device HEXABITZ_ICs:MAX30100EFD+ -> HEXABITZ_ICs:MAX30101EFD+T
Connections:
- removed net +1V8: C10.+, C9.1, U2.OUT, U3.VDD
- removed net USART6_RX: P1.SD1, U1.PB9
- removed net USART6_TX: P1.SU1, U1.PB8
- new net +1.8V: C12.1, C8.1, C9.1, U2.OUT, U3.VDD
- new net +5V: C10.1, C11.1, R10.2, R7.2, U4.OUT
- new net N$12: L1.2, U4.LX
- new net N$9: C11.2, R7.1, R8.2, U4.FB
- net GND: now also C10.2, C13.2, C14.2, C7.2, D2.A, R8.1, U4.GND; no longer C10.-, C11.-, C7.-, U1.EPAD, U1.PA15, U1.PB6, U1.PB7, U1.PC13, U1.PC14-OSC32_IN, U1.PD0, U3.PGND
- net INT: now also R6.1, U1.PB7; no longer INT.P$1, R4.1, U1.PD1
- net N$1: now also U1.PB13; no longer U1.PA5
- net N$2: now also C5.1, C7.1, R10.1, R9.1, U3.VLED+; no longer C12.1, U2.BYPASS
- net SCL: now also R4.1; no longer R5.1, SCL.P$1
- net SDA: now also R5.1; no longer R6.1, SDA.P$1
- net USART4_RX: now also P1.SD1
- net USART4_TX: now also P1.SU1
- net VDD: now also C13.1, C14.1, D2.C, L1.1, R9.2, U2.EN, U4.EN, U4.VIN; no longer C11.+, C5.1, C7.+, C8.1, U1.VDDIO2, U2.INHIBIT, U3.IR_LED+, U3.R_LED+
- net VDDA: now also C2.1, C4.1; no longer C2.+, C4.+
- net VSSA: now also C2.2, C4.2; no longer C2.-, C4.-
Other:
- note added: "1.8V LDO Reguletor"
- note added: "Boost Converter"
- note added: "H2BR1"
- note added: "H2BR1_Backend"
- note added: "H2BR1_Frontend"
- note removed: "0"
- note removed: "H2BR10"
- note removed: "H2BR10_Backend"
- note removed: "H2BR10_Frontend"
- note removed: "Obada Albasha"
- note removed: "VDDIO2 Coupling"
- moved on the sheet: C12, C8, C9, D1, R1, R4, R5, R6
